Commit message: nanocar_bug

File: data/nanocarpro/urdf/nanocarpro.urdf (robot description, URDF)
Before this commit: robot NanoCarPro, 12 links, 11 joints
Links:
- removed link /base_link
- added link base_link, mass 0.45437; collision box size=0.21 0.1 0.095; visual mesh filename=../meshes/base_link.obj
Joints:
- joint back_left_wheel_joint: parent /base_link -> base_link
- joint back_right_wheel_joint: parent /base_link -> base_link
- joint base_joint: child /base_link -> base_link
- joint camera_joint: parent /base_link -> base_link
- joint imu_joint: parent /base_link -> base_link
- joint ir_camera_joint: parent /base_link -> base_link
- joint laser_joint: parent /base_link -> base_link
- joint left_steering_joint: parent /base_link -> base_link
- joint right_steering_joint: parent /base_link -> base_link

Commit message: adjust urdf

File: data/nanocarpro/urdf/nanocarpro.urdf (robot description, URDF)
Before this commit: robot NanoCarPro, 12 links, 11 joints
Links:
- removed link /base_footprint
- added link base
Joints:
- joint base_joint: parent /base_footprint -> base
- joint left_steering_joint: limit (none) -> lower=-0.7854 upper=0.7854 effort=30 velocity=2.0; type continuous -> revolute
- joint right_steering_joint: limit (none) -> lower=-0.7854 upper=0.7854 effort=30 velocity=2.0; type continuous -> revolute
